File: Wand/Wand.sch (KiCad schematic (older format))
At the start: 28 parts, among them IC1 ATMEGA328-MMH, J1 ACJS-NH35, P1 ISP, P2 BASE, U1 OPA336U, U2 MPU-6050, Y1 16MHz

Commit message: General tidy-up and added a 100nF cap on AREF.
Parts:
- added C9: 100n, Capacitors_SMD:C_0402, symbol C
- C1, C2, C3, C4: footprint (none) -> Capacitors_SMD:C_0402
- C5, C7: value 0.1uF -> 100n; footprint (none) -> Capacitors_SMD:C_0402
- C6: value 10nF -> 10n; footprint (none) -> Capacitors_SMD:C_0402
- C8: value 2.2nF -> 2.2n; footprint (none) -> Capacitors_SMD:C_0402
- R1, R11, R2, R3, R4, R5, R6, R7, R8: footprint (none) -> Resistors_SMD:R_0402
- R10, R9: value 10K -> 10k; footprint (none) -> Resistors_SMD:R_0402
- U3: renamed from IC1; footprint TQFP32 -> (none)
- gave numbers to parts that had none: 1
- renumbered J1 to P3
Connections:
- wire segments 117 -> 119
Other:
- moved on the sheet: C2, C4, C5, C6, C7, C8, D1, P1, P2, P3, R10, R11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

Commit message: Updated the Op-amp for the smaller OPA336N version
Parts:
- U1: value OPA336U -> OPA336N
Changed lines of the file:
@@
 P 3400 6350
 F 0 "U1" H 3550 6650 70  0000 C CNN
-F 1 "OPA336U" H 3550 6550 70  0000 C CNN
+F 1 "OPA336N" H 3550 6550 70  0000 C CNN
 F 2 "" H 3400 6350 60  0001 C CNN
 F 3 "" H 3400 6350 60  0000 C CNN

Commit message: Added a few footprints
Parts:
- P1: footprint (none) -> Wand:ISP_pads_2x3
- U1: footprint (none) -> Wand:OPA336_Plastic_Small; symbol TL071 -> TL071-RESCUE-Wand
- U2: footprint (none) -> Wand:MPU-6050
Changed lines of the file:
@@
 EESchema Schematic File Version 2
+LIBS:Wand-rescue
 LIBS:power
 LIBS:device
@@
 F 0 "U2" H 8000 1600 60  0000 C CNN
 F 1 "MPU-6050" H 7400 1600 60  0000 C CNN
-F 2 "" H 7650 2050 60  0001 C CNN
+F 2 "Wand:MPU-6050" H 7650 2050 60  0001 C CNN
 F 3 "" H 7650 2050 60  0000 C CNN
 	1    7650 2300
@@
 $EndComp
 $Comp
-L TL071 U1
+L TL071-RESCUE-Wand U1
 U 1 1 56411DEC
 P 3400 6350
 F 0 "U1" H 3550 6650 70  0000 C CNN
 F 1 "OPA336N" H 3550 6550 70  0000 C CNN
-F 2 "" H 3400 6350 60  0001 C CNN
+F 2 "Wand:OPA336_Plastic_Small" H 3400 6350 60  0001 C CNN
 F 3 "" H 3400 6350 60  0000 C CNN
 	1    3400 6350
@@
 F 0 "P1" H 9950 3850 50  0000 C CNN
 F 1 "ISP" H 9950 3450 50  0000 C CNN
-F 2 "" H 9950 2450 60  0001 C CNN
+F 2 "Wand:ISP_pads_2x3" H 9950 2450 60  0001 C CNN
 F 3 "" H 9950 2450 60  0000 C CNN
 	1    9950 3650

Commit message: Corrected the schematic to use the 28pin version of the ATMEGA 328
Parts:
- U3: symbol ATMEGA328P-A -> ATMEGA328P-MM
Connections:
- wire segments 119 -> 117
- no-connect marks 15 -> 13
Changed lines of the file:
@@
 EESchema Schematic File Version 2
-LIBS:Wand-rescue
 LIBS:power
 LIBS:device
@@
 $EndDescr
 $Comp
-L ATMEGA328P-A U3
-U 1 1 563E7654
-P 2450 2550
-F 0 "U3" H 1700 3800 40  0000 L BNN
-F 1 "ATMEGA328-MMH" H 2850 1150 40  0000 L BNN
-F 2 "" H 2450 2550 30  0000 C CIN
-F 3 "" H 2450 2550 60  0000 C CNN
-	1    2450 2550
-	1    0    0    -1
-$EndComp
-$Comp
 L Crystal Y1
 U 1 1 563E76C3
@@
 Text Label 3600 3650 0    60   ~ 0
 LED_B
-NoConn ~ 1550 2800
-NoConn ~ 1550 2900
 NoConn ~ 3450 3750
 NoConn ~ 3450 3450
@@
 Wire Wire Line
 	1300 2050 1550 2050
-Connection ~ 1300 1550
 Wire Wire Line
 	1300 1750 1550 1750
@@
 Wire Wire Line
 	9650 5250 9450 5250
-Connection ~ 1400 3650
-Wire Wire Line
-	1550 3550 1400 3550
-Connection ~ 1400 3750
 Wire Wire Line
 	1400 3650 1550 3650
 Wire Wire Line
 	1400 3750 1550 3750
-Wire Wire Line
-	1400 3550 1400 3900
 Connection ~ 1300 1450
-Wire Wire Line
-	1300 1550 1550 1550
 Wire Wire Line
 	1300 1450 1550 1450
@@
 Wire Wire Line
 	1300 2050 1300 2100
+$Comp
+L ATMEGA328P-MM U3
+U 1 1 563E7654
+P 2450 2550
+F 0 "U3" H 1700 3800 40  0000 L BNN
+F 1 "ATMEGA328-MMH" H 2850 1150 40  0000 L BNN
+F 2 "" H 2450 2550 30  0000 C CIN
+F 3 "" H 2450 2550 60  0000 C CNN
+	1    2450 2550
+	1    0    0    -1
+$EndComp
+Wire Wire Line
+	1400 3650 1400 3900
 $EndSCHEMATC

Commit message: Footprint for ATMega328-MM
Parts:
- U3: footprint (none) -> Wand:QFN-28-1EP_4x4mm_Pitch0.45mm
Changed lines of the file:
@@
 F 0 "U3" H 1700 3800 40  0000 L BNN
 F 1 "ATMEGA328-MMH" H 2850 1150 40  0000 L BNN
-F 2 "" H 2450 2550 30  0000 C CIN
+F 2 "Wand:QFN-28-1EP_4x4mm_Pitch0.45mm" H 2450 2550 30  0001 C CIN
 F 3 "" H 2450 2550 60  0000 C CNN
 	1    2450 2550

Commit message: Added footprint for the LED
Parts:
- D1: footprint (none) -> Wand:Tri-Colour_LED
- U4: footprint (none) -> TO_SOT_Packages_SMD:SOT-23-6
Changed lines of the file:
@@
 F 0 "D1" H 5650 5500 50  0000 C CNN
 F 1 "ASMB-MTB0-0A3A2" H 5650 4800 50  0000 C CNN
-F 2 "" H 5605 5100 50  0001 C CNN
+F 2 "Wand:Tri-Colour_LED" H 5605 5100 50  0001 C CNN
 F 3 "" H 5605 5100 50  0000 C CNN
 	1    5650 5150
@@
 F 0 "U4" H 7350 5350 60  0000 C CNN
 F 1 "TMP100" H 7350 4750 60  0000 C CNN
-F 2 "" H 7350 5050 60  0001 C CNN
+F 2 "TO_SOT_Packages_SMD:SOT-23-6" H 7350 5050 60  0001 C CNN
 F 3 "" H 7350 5050 60  0000 C CNN
 	1    7350 5050

Commit message: Changed 3.5mm jack to an EBS35 style jack as a) I have some and b) some one had already done the footprint
Parts:
- P2: footprint (none) -> Pin_Headers:Pin_Header_Straight_1x05
- P3: value ACJS-NH35 -> EBS35; symbol JACK_TRS_6PINS -> REICHELT_EBS35
Connections:
- net GND: now also P3.3 (Sleeve), R11.1; no longer P3.1 (S), R11.2
- net HEAT: now also P3.1 (Tip); no longer P3.3 (R)
- net TIP_DETECT: now also P3.4 (TipSwitch), R11.2; no longer P3.5 (TN), R11.1
- no-connect marks 13 -> 12
Other:
- moved on the sheet: R11
Changed lines of the file:
@@
 LIBS:Wand
 LIBS:tmp10x
+LIBS:EBS35
 LIBS:Wand-cache
 EELAYER 25 0
@@
 $EndComp
 $Comp
-L JACK_TRS_6PINS P3
+L REICHELT_EBS35 P3
 U 1 1 56411635
-P 10050 5050
-F 0 "P3" H 10050 5450 50  0000 C CNN
-F 1 "ACJS-NH35" H 10000 4750 50  0000 C CNN
-F 2 "" H 10150 4900 60  0001 C CNN
-F 3 "" H 10150 4900 60  0000 C CNN
-	1    10050 5050
-	-1   0    0    1
+P 10250 5100
+F 0 "P3" H 10250 5500 50  0000 C CNN
+F 1 "EBS35" H 10200 4800 50  0000 C CNN
+F 2 "" H 10350 4950 60  0001 C CNN
+F 3 "" H 10350 4950 60  0000 C CNN
+	1    10250 5100
+	1    0    0    -1
 $EndComp
 $Comp
@@
 L GND #PWR06
 U 1 1 56416557
-P 9450 5500
-F 0 "#PWR06" H 9450 5250 50  0001 C CNN
-F 1 "GND" H 9450 5350 50  0000 C CNN
-F 2 "" H 9450 5500 60  0000 C CNN
-F 3 "" H 9450 5500 60  0000 C CNN
-	1    9450 5500
-	1    0    0    -1
-$EndComp
-Text Label 9450 5050 2    60   ~ 0
+P 9350 5050
+F 0 "#PWR06" H 9350 4800 50  0001 C CNN
+F 1 "GND" H 9350 4900 50  0000 C CNN
+F 2 "" H 9350 5050 60  0000 C CNN
+F 3 "" H 9350 5050 60  0000 C CNN
+	1    9350 5050
+	0    1    1    0
+$EndComp
+Text Label 9450 4950 2    60   ~ 0
 SENS
 Text Label 9450 4850 2    60   ~ 0
@@
 F 0 "P2" H 10200 2200 50  0000 C CNN
 F 1 "BASE" V 10300 1900 50  0000 C CNN
-F 2 "" H 10200 1900 60  0001 C CNN
+F 2 "Pin_Headers:Pin_Header_Straight_1x05" H 10200 1900 60  0001 C CNN
 F 3 "" H 10200 1900 60  0000 C CNN
 	1    10200 1900
@@
 	-1   0    0    1
 $EndComp
-NoConn ~ 9650 4950
-NoConn ~ 9650 5350
+NoConn ~ 9650 5300
 $Comp
 L +3.3V #PWR011
@@
 	1    0    0    -1
 $EndComp
-Text Label 9150 5150 2    60   ~ 0
+Text Label 9350 5350 2    60   ~ 0
 TIP_DETECT
 $Comp
 L R R11
 U 1 1 564A6CD4
-P 9300 5300
-F 0 "R11" V 9380 5300 50  0000 C CNN
-F 1 "2M" V 9300 5300 50  0000 C CNN
-F 2 "Resistors_SMD:R_0402" V 9230 5300 30  0001 C CNN
-F 3 "" H 9300 5300 30  0000 C CNN
-	1    9300 5300
+P 9450 5200
+F 0 "R11" V 9530 5200 50  0000 C CNN
+F 1 "2M" V 9450 5200 50  0000 C CNN
+F 2 "Resistors_SMD:R_0402" V 9380 5200 30  0001 C CNN
+F 3 "" H 9450 5200 30  0000 C CNN
+	1    9450 5200
 	1    0    0    -1
 $EndComp
@@
 	9650 4850 9450 4850
 Wire Wire Line
-	9450 5050 9650 5050
-Wire Wire Line
-	9650 5250 9450 5250
+	9450 4950 9650 4950
 Wire Wire Line
 	1400 3650 1550 3650
@@
 Wire Wire Line
 	1150 6250 1750 6250
-Wire Wire Line
-	9450 5250 9450 5500
-Connection ~ 9450 5450
-Wire Wire Line
-	9450 5450 9300 5450
-Wire Wire Line
-	9150 5150 9650 5150
-Connection ~ 9300 5150
 Text Notes 8700 5850 0    60   ~ 0
 SENS pulled high (3.3v) with 1M resister
@@
 Wire Wire Line
 	1400 3650 1400 3900
+Wire Wire Line
+	9350 5350 9600 5350
+Wire Wire Line
+	9600 5350 9600 5200
+Wire Wire Line
+	9600 5200 9650 5200
+Connection ~ 9450 5350
+Wire Wire Line
+	9350 5050 9650 5050
+Connection ~ 9450 5050
 $EndSCHEMATC

Commit message: Set the footprint of the 3.5mm socket
Parts:
- P3: footprint (none) -> Wand:Reichelt_EBS35
Changed lines of the file:
@@
 F 0 "P3" H 10250 5500 50  0000 C CNN
 F 1 "EBS35" H 10200 4800 50  0000 C CNN
-F 2 "" H 10350 4950 60  0001 C CNN
+F 2 "Wand:Reichelt_EBS35" H 10350 4950 60  0001 C CNN
 F 3 "" H 10350 4950 60  0000 C CNN
 	1    10250 5100
